Commit message: feat(sim): single-source kinematics params from URDF (#8)
wheel_radius / wheel_separation / laser_x 此前在 URDF 与 sim_params.yaml
两处手工同步（且 URDF 根本没有轮，数值实际只存在于 yaml，TF 链与仿真
真值靠人肉核对）。改为 URDF 单一事实源：

- mining_truck.urdf 增加 wheel_left/right（cylinder r=0.10，joint y=±0.21，
  名称对齐 sim 发布的 /joint_states；continuous 类型让 rsp 用真实转角发轮 TF）；
- 新增纯 Python 解析器 urdf_kinematics.py（stdlib ElementTree，无新依赖，
  5 例单测，含对真实 URDF 的对拍）；
- sim 节点启动时解析 URDF（urdf_file 参数，默认定位 smart_charge_base
  包内文件），成功则以 URDF 值覆盖 yaml fallback 并 log，失败 warn 回退；
  里程计积分改用缓存值（原每 tick get_parameter，且与事实源脱节）。

容器内已验证：节点启动 log「运动学参数来自 URDF（单一事实源）:
wheel_radius=0.1, wheel_separation=0.42, laser_x=0.15」。数值零变化，
纯结构重构。runtime ros2 param set laser_x 仍可作为操作员显式覆盖。

Co-Authored-By: Claude Opus 5 <noreply@anthropic.com>

File: src/smart_charge_base/urdf/mining_truck.urdf (robot description, URDF)
Before this commit: robot smart_charge_mining_truck, 3 links, 2 joints
Links:
- added link wheel_left; visual cylinder length=0.04 radius=0.10
- added link wheel_right; visual cylinder length=0.04 radius=0.10
Joints:
- added joint left_wheel_joint: type continuous, parent base_link, child wheel_left, origin xyz=0.0 0.21 0.10, axis 0 1 0
- added joint right_wheel_joint: type continuous, parent base_link, child wheel_right, origin xyz=0.0 -0.21 0.10, axis 0 1 0
